File: lv/kicad-template/template.kicad_sch (KiCad schematic)
At the start: 0 parts

Commit message: Testing commit
Hi
Parts:
- added C1: 10nF, Capacitor_SMD:C_0603_1608Metric, symbol Device:C_Small
- added D1: D_Small, Diode_SMD:D_0201_0603Metric, symbol Device:D_Small
- added J1: TS_IN, Connector_PinHeader_2.54mm:PinHeader_1x02_P2.54mm_Vertical, symbol Connector_Generic:Conn_01x02
- added J2: PK_HOLD_OUT, Connector_PinHeader_2.54mm:PinHeader_1x05_P2.54mm_Vertical_SMD_Pin1Left, symbol Connector_Generic:Conn_01x02
- added R1: 24k, Resistor_SMD:R_0603_1608Metric, symbol Device:R_Small
- added R2: 1k, Resistor_SMD:R_0603_1608Metric, symbol Device:R_Small
- added U1: MCP6004, Package_SO:SOIC-14_3.9x8.7mm_P1.27mm, symbol Amplifier_Operational:MCP6004
Connections:
- new net: D1.2 (A), U1.1
- new net: R1.2, R2.1, U1.3 (+)
- new net: J2.1 (Pin_1), U1.6 (-), U1.7
- new net GND: C1.2, J1.1 (Pin_1), J2.2 (Pin_2), R2.2
- new net PK_HOLD_VAL: C1.1, D1.1 (K), U1.2 (-), U1.5 (+)
- new net TS+: J1.2 (Pin_2), R1.1
Other:
- note added: "TS-"
