File: pe/zander-hong/template.kicad_sch (KiCad schematic)
At the start: 0 parts

Commit message: schematic finished
Parts:
- added C1, C2, C2A, C3: C, symbol Device:C
- added L1: L, symbol Device:L
- added R1, R2: R, symbol Device:R
- added U1: AP62300TWU, Package_TO_SOT_SMD:TSOT-23-6, symbol Regulator_Switching:AP62300TWU
Connections:
- new net: R1.1, R2.1, U1.4 (FB)
- new net: C3.1, L1.2, U1.2 (SW)
- new net: C3.2, U1.6 (BST)
- new net +12V: C1.2, U1.3 (IN), U1.5 (EN)
- new net GND: C1.1, C2.1, C2A.2, R2.2, U1.1 (GND)
- new net Vout: C2.2, C2A.1, L1.1, R1.2
Other:
- note added: "C1: Input Filtering Cap C2 & C2A: Output Filtering Cap in parrallel to account for DC Bias Derating C3: Bootstrap Cap to power gate for N channel MOSFET"
- note added: "R1 & R2: Sample Voltage Output to ensure precise step down"
