File: pe/timmy-li/buck1.kicad_sch (KiCad schematic)
At the start: 5 parts, among them U1 TPS62143

Commit message: broken
Parts:
- added C3: 3.3nF, Capacitor_SMD:C_0201_0603Metric_Pad0.64x0.40mm_HandSolder, symbol Device:C_Small
Connections:
- net GND: now also C3.2; no longer U1.9 (SS/TR)
- new net: C3.1, U1.9 (SS/TR)
Other:
- note added: "5-17V"
- note added: "5V/2A"
