File: pe/timmy-li/buck1.kicad_pcb (KiCad board)
At the start: 2 copper layers, 5 parts, among them U1 TPS62143

Commit message: broken
Parts:
- removed C1: 10uF, Capacitor_SMD:C_0201_0603Metric_Pad0.64x0.40mm_HandSolder
- removed C2: 22uF, Capacitor_SMD:C_0201_0603Metric_Pad0.64x0.40mm_HandSolder
- removed L1: 2.2uH, Inductor_SMD:L_1210_3225Metric_Pad1.42x2.65mm_HandSolder
- removed R1: 100k, Resistor_SMD:R_0603_1608Metric
- removed U1: TPS62143, Package_DFN_QFN:VQFN-16-1EP_3x3mm_P0.5mm_EP1.68x1.68mm_ThermalVias

Commit message: Update buck1.kicad_pcb
Parts:
- added C1: 10uF, Capacitor_SMD:C_0201_0603Metric_Pad0.64x0.40mm_HandSolder, F.Cu at (111.0, 102.6)
- added C2: 22uF, Capacitor_SMD:C_0201_0603Metric_Pad0.64x0.40mm_HandSolder, F.Cu at (119.5, 102.9)
- added C3: 3.3nF, Capacitor_SMD:C_0201_0603Metric_Pad0.64x0.40mm_HandSolder, F.Cu at (112.0, 102.6)
- added L1: 2.2uH, Inductor_SMD:L_1210_3225Metric_Pad1.42x2.65mm_HandSolder, F.Cu at (114.5, 99.0)
- added R1: 100k, Resistor_SMD:R_0603_1608Metric, F.Cu at (118.0, 102.7)
- added U1: TPS62143, Package_DFN_QFN:VQFN-16-1EP_3x3mm_P0.5mm_EP1.68x1.68mm_ThermalVias, F.Cu at (114.7, 102.9)
