File: pe/timmy-li/_restore_backup_2026-10-11T21-27-11-198/template.kicad_sch (KiCad schematic)
At the start: 5 parts, among them U1 TPS62143

Commit message: broken
Parts:
- removed V1: 13.5, symbol Simulation_SPICE:VDC
- added C3: 3.3nf, Capacitor_SMD:C_0201_0603Metric_Pad0.64x0.40mm_HandSolder, symbol Device:C_Small
- added R1: 100k, Resistor_SMD:R_0201_0603Metric_Pad0.64x0.40mm_HandSolder, symbol Device:R
- C1, C2: footprint (none) -> Capacitor_SMD:C_0201_0603Metric_Pad0.64x0.40mm_HandSolder
- L1: footprint (none) -> Inductor_SMD:L_0603_1608Metric_Pad1.05x0.95mm_HandSolder
Connections:
- net GND: now also C2.2, U1.5 (FB)
- net at L1.2: now also C2.1, U1.14 (VOS), R1.1
- net at C1.2: now also C3.2; no longer U1.9 (SS/TR)
- net at U1.4 (PG): now also R1.2
- new net: C3.1, U1.9 (SS/TR)
Other:
- moved on the sheet: C2
