File: lv/maheer-grang/maheer-grang.kicad_sch (KiCad schematic)
At the start: 0 parts

Commit message: finished lv project research, working on lv board schematic. worked on pe buck schematic
Other:
- title: ${BOARD_TITLE} -> LV Driver Audio Onboarding Project
Changed lines of the file:
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@@
 	(paper "A")
 	(title_block
-		(title "${BOARD_TITLE}")
+		(title "LV Driver Audio Onboarding Project")
 		(date "${CURRENT_DATE}")
 		(rev "${REVISION}")
 		(company "Formula Slug")
-		(comment 1 "${NAMES}")
+		(comment 1 "Maheer Grang")
 		(comment 2 "${COMMENT1}")
 		(comment 3 "${COMMENT2}")
