File: pe/madison-patiag/madison-patiag.kicad_sch (KiCad schematic)
At the start: 0 parts

Commit message: feat: initial buck converter wiring
Parts:
- added C_{BOOT}1, C_{in}2: 0.1uF, symbol Device:C
- added C_{in}1, C_{out}1, C_{out}2: 22uF, symbol Device:C
- added L1: 8.2uH, symbol Device:L
- added R1: 105k, SOIC_5EHGJ8F_RIT, symbol Device:R_US
- added R2: 20k, SOIC_5EHGJ8F_RIT, symbol Device:R_US
- added R3: 20, SOIC_5EHGJ8F_RIT, symbol Device:R_US
- added R4: 100k, SOIC_5EHGJ8F_RIT, symbol Device:R_US
- added U1: RT6215EHGJ8F, SOIC_5EHGJ8F_RIT, symbol 2026-10-08_19-50-54:RT6215EHGJ8F
Connections:
- new net: R4.1, U1.1 (MODE)
- new net: C_{BOOT}1.2, L1.1, U1.3 (SW)
- new net: R3.1, U1.5 (BOOT)
- new net: R1.1, R2.2, U1.8 (FB)
- new net: C_{BOOT}1.1, R3.2
- new net +12V: C_{in}1.1, C_{in}2.1, R4.2, U1.2 (VIN), U1.6 (EN)
- new net +5V: C_{out}1.1, C_{out}2.1, L1.2, R1.2
- new net GND: C_{in}1.2, C_{in}2.2, C_{out}1.2, C_{out}2.2, R2.1, U1.4 (GND)

Commit message: feat: add footprints to all components
Parts:
- added C_{out}3: 22uF, Capacitor_SMD:C_0603_1608Metric_Pad1.08x0.95mm_HandSolder, symbol Device:C
- C_{BOOT}1, C_{in}2, C_{out}1, C_{out}2: footprint (none) -> Capacitor_SMD:C_0603_1608Metric_Pad1.08x0.95mm_HandSolder
- C_{in}1: footprint (none) -> Capacitor_SMD:C_1206_3216Metric_Pad1.33x1.80mm_HandSolder
- L1: footprint (none) -> Inductor_SMD:L_Taiyo-Yuden_MD-4040
- R1, R2, R3, R4: footprint SOIC_5EHGJ8F_RIT -> Resistor_SMD:R_0603_1608Metric_Pad0.98x0.95mm_HandSolder
- U1: footprint SOIC_5EHGJ8F_RIT -> Package_TO_SOT_SMD:TSOT-23-8_HandSoldering
Connections:
- net +5V: now also C_{out}3.1
- net GND: now also C_{out}3.2

Commit message: feat: updated PCB and added initial traces
Changed lines of the file:
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@@
+	)
+	(junction
+		(at 87.63 67.31)
+		(diameter 0)
+		(color 0 0 0 0)
 	)
 	(junction
@@
 	(wire
 		(pts
+			(xy 87.63 67.31) (xy 87.63 68.58)
+		)
+		(stroke
+			(width 0)
+			(type default)
+		)
+	)
+	(wire
+		(pts
 			(xy 50.8 41.91) (xy 64.77 41.91)
 		)
@@
 	(wire
 		(pts
-			(xy 87.63 64.77) (xy 87.63 68.58)
+			(xy 87.63 64.77) (xy 87.63 67.31)
 		)
 		(stroke
@@
 					(unit 1)
 				)
+			)
+		)
+	)
+	(symbol
+		(lib_id "power:PWR_FLAG")
+		(at 87.63 67.31 270)
+		(unit 1)
+		(body_style 1)
+		(exclude_from_sim no)
+		(in_bom yes)
+		(on_board yes)
+		(in_pos_files yes)
+		(dnp no)
+		(property "Reference" "#FLG03"
+			(at 89.535 67.31 0)
+			(hide yes)
+			(show_name no)
+			(do_not_autoplace no)
+			(effects
+				(font
+					(size 1.27 1.27)
+				)
+			)
+		)
+		(property "Value" "PWR_FLAG"
+			(at 91.44 67.564 0)
+			(show_name no)
+			(do_not_autoplace no)
+			(effects
+				(font
+					(size 1.27 1.27)
+				)
+			)
+		)
+		(property "Footprint" ""
+			(at 87.63 67.31 0)
+			(hide yes)
+			(show_name no)
+			(do_not_autoplace no)
+			(effects
+				(font
+					(size 1.27 1.27)
+				)
+			)
+		)
+		(property "Datasheet" ""
+			(at 87.63 67.31 0)
+			(hide yes)
+			(show_name no)
+			(do_not_autoplace no)
+			(effects
+				(font
+					(size 1.27 1.27)
+				)
+			)
+		)
+		(property "Description" "Special symbol for telling ERC where power comes from"
+			(at 87.63 67.31 0)
+			(hide yes)
+			(show_name no)
+			(do_not_autoplace no)
+			(effects
+				(font
+					(size 1.27 1.27)
+				)
+			)
+		)
+		(pin "1"
+		)
+		(instances
+			(project "madison-patiag"
+				(path "/e994741c-7c7d-4124-9d00-43b883baa61d"
+					(reference "#FLG03")
+					(unit 1)
+				)
