File: pe/madison-patiag/madison-patiag.kicad_pcb (KiCad board)
At the start: 2 copper layers, 12 parts, among them U1 RT6215EHGJ8F

Commit message: feat: finished PCB with no errors or warnings, needs review
Other:
- board outline added: 13.2 x 11.9 mm
Changed lines of the file:
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@@
 		(capping no)
 		(filling no)
+		(zone_defaults)
 		(pcbplotparams
 			(layerselection 0x00000000_00000000_55555555_5755f5ff)
@@
 		(tags "capacitor handsolder")
 		(property "Reference" "C_{in}1"
-			(at 3.7 -0.5 90)
-			(layer "F.SilkS")
-			(effects
-				(font
-					(size 0.7 0.7)
-					(thickness 0.15)
+			(at 3.2625 0 180)
+			(layer "F.SilkS")
+			(effects
+				(font
+					(size 1.016 0.7)
+					(thickness 0.1524)
+					(bold yes)
 				)
 			)
@@
 			(at 3.6 0.4 90)
 			(layer "F.Fab")
+			(hide yes)
 			(effects
 				(font
@@
 			(at -4.5 0 90)
 			(layer "F.Fab")
+			(hide yes)
 			(effects
 				(font
@@
 		)
 		(fp_text user "${REFERENCE}"
-			(at -2.6 0 90)
+			(at -1.8 0 180)
 			(layer "F.Fab")
 			(effects
@@
 			(effects
 				(font
-					(size 1 1)
-					(thickness 0.15)
+					(size 1.016 1)
+					(thickness 0.1524)
 				)
 			)
@@
 			(at 0 2.8 0)
 			(layer "F.Fab")
+			(hide yes)
 			(effects
 				(font
@@
 			(at -2.5 -0.015 0)
 			(layer "F.Fab")
+			(hide yes)
 			(effects
 				(font
@@
 			(at 0.1 1.2 90)
 			(layer "F.Fab")
+			(hide yes)
 			(effects
 				(font
@@
 		(tags "capacitor handsolder")
 		(property "Reference" "C_{in}2"
-			(at 2.8 -0.4 90)
-			(layer "F.SilkS")
-			(effects
-				(font
-					(size 0.7 0.7)
-					(thickness 0.15)
+			(at 2.7625 0.5 90)
+			(layer "F.SilkS")
+			(effects
+				(font
+					(size 1.016 0.7)
+					(thickness 0.1524)
+					(bold yes)
 				)
 			)
@@
 			(at 2.8 0.5 90)
 			(layer "F.Fab")
+			(hide yes)
 			(effects
 				(font
@@
 			(at -2.7 0 0)
 			(layer "F.Fab")
+			(hide yes)
 			(effects
 				(font
@@
 			(at -2.8625 -0.3 0)
 			(layer "F.Fab")
+			(hide yes)
 			(effects
 				(font
@@
 		)
 		(fp_text user "${REFERENCE}"
-			(at -2.8625 0.4 0)
+			(at -0.0625 1 0)
 			(layer "F.Fab")
 			(effects
@@
 			(at -4.5 0 90)
 			(layer "F.Fab")
+			(hide yes)
 			(effects
 				(font
@@
 		)
 		(fp_text user "${REFERENCE}"
-			(at -2.6 0 90)
+			(at -1.8 0 180)
 			(layer "F.Fab")
 			(effects
@@
 			(at 0.0125 -1.3 0)
 			(layer "F.Fab")
+			(hide yes)
 			(effects
 				(font
@@
 			(at -4.5 0.01 90)
 			(layer "F.Fab")
+			(hide yes)
 			(effects
 				(font
@@
 		)
 		(fp_text user "${REFERENCE}"
-			(at -2.5 -0.09 90)
+			(at -1.8 0.01 180)
 			(layer "F.Fab")
 			(effects
@@
 			)
 		)
+	)
+	(gr_rect
+		(start 137.3 104)
+		(end 150.5 115.9)
+		(stroke
+			(width 0.0508)
+			(type default)
+		)
+		(fill no)
+		(layer "Edge.Cuts")
 	)
 	(segment
@@
 		(layer "F.Cu")
 		(net "+12V")
-	)
-	(segment
-		(start 144.8 109.646)
-		(end 144.7 109.746)
-		(width 0.5)
-		(layer "F.Cu")
-		(net "+12V")
