File: pe/benjamin-rogoff.kicad_sch (KiCad schematic)
At the start: 8 parts

Commit message: Add files via upload
Updated Circuit
Parts:
- BuckConverter: Digi PN (none) -> 497-DCP3603ACMRTR-ND; Digi URL (none) -> https://www.digikey.com/en/products/detail/stmicroelectroni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; MFG (none) -> STMicroelectronics; MFG PN (none) -> DCP3603ACMR
- C_Boot: Digi PN (none) -> 399-C0603C104M5RACTUTR-ND; Digi URL (none) -> https://www.digikey.com/en/products/detail/kemet/C0603C104M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; MFG (none) -> KEMET; MFG PN (none) -> C0603C104M5RACTU
- Cin: Digi PN (none) -> 587-4967-2-ND; Digi URL (none) -> https://www.digikey.com/en/products/detail/taiyo-yuden/UMK3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; MFG (none) -> Taiyo Yuden; MFG PN (none) -> UMK316B7225ML-T
- Cout1, Cout2: Digi PN (none) -> 4713-GMC31X5R226M25NTTR-ND; Digi URL (none) -> https://www.digikey.com/en/products/detail/cal-chip-electro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; MFG (none) -> Cal-Chip Electronics, Inc.; MFG PN (none) -> GMC31X5R226M25NT
- L: renamed from L1; value L -> 6.8uH; Digi PN (none) -> 553-BWVS006060456R8M00TR-ND; Digi URL (none) -> https://www.digikey.com/en/products/detail/pulse-electronic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; MFG (none) -> Pulse Electronics; MFG PN (none) -> BWVS006060456R8M00
- R1: value R -> 73.2kΩ
- R2: value R -> 15kΩ
