File: pe/Buck_Conv_Final/Buck_Final.kicad_pcb (KiCad board)
At the start: 2 copper layers, 10 parts, among them U2 TPS5405DR

Commit message: Library for buck IC, math for components, minor updates
Parts:
- added Vin1: Conn_01x02, Connector_PinHeader_1.00mm:PinHeader_1x02_P1.00mm_Vertical, F.Cu at (102.0, 99.5)
- added Vout1: ~, Connector_PinHeader_1.00mm:PinHeader_1x02_P1.00mm_Vertical, F.Cu at (111.0, 99.5)
