File: pe/timmy-li/actual sch and pcb/buck1.kicad_sch (KiCad schematic)
At the start: 6 parts, among them U1 TPS62143

Commit message: added labels
Connections:
- net Output 5V/2A: now reaches C2.1, L1.2, R1.1, U1.14 (VOS)
- net Input 5-17V: now reaches C1.1, U1.10 (VIN), U1.11 (VIN), U1.12 (VIN), U1.13 (EN)
Other:
- note removed: "5-17V"

Commit message: added symbol fields
Parts:
- C1: Digikey Part Number (none) -> 311-3494-2-ND; Digikey URL (none) -> https://www.digikey.com/en/products/detail/yageo/CC0603MRX5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; Manufacturer (none) -> YAGEO; Manufacturer Part Number (none) -> CC0603MRX5R8BB106
- C2: Digikey Part Number (none) -> 6639-MH0603A226M100N8RCZATR-ND; Digikey URL (none) -> https://www.digikey.com/en/products/detail/sunway-communica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; Manufacturer (none) -> Sunway Communication; Manufacturer Part Number (none) -> MH0603A226M100N8RCZA
- L1: Digikey Part Number (none) -> 595-F1C1-322510-2R2MTR-ND; Digikey URL (none) -> https://www.digikey.com/en/products/detail/signal-transform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; Manufacturer (none) -> Signal Transformer; Manufacturer Part Number (none) -> F1C1-322510-2R2M
Other:
- note removed: "5V/2A"
Changed lines of the file:
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@@
 		(comment 3 "${COMMENT2}")
-	)
-	(text "5V/2A"
-		(exclude_from_sim no)
-		(at 140.208 74.676 0)
-		(effects
-			(font
-				(size 1.27 1.27)
-			)
-		)
 	)
 	(junction
@@
 			)
 		)
-		(property "Datasheet" ""
+		(property "Datasheet" "https://belfuse.com/media/datasheets/products/chokes-coils-inductors/ds-ST-F1C1-3225-series.pdf"
 			(at 115.57 78.74 0)
 			(hide yes)
@@
 			)
 		)
-		(property "Digikey Part Number" ""
+		(property "Digikey Part Number" "595-F1C1-322510-2R2MTR-ND"
 			(at 115.57 78.74 0)
 			(hide yes)
@@
 			)
 		)
-		(property "Digikey URL" ""
+		(property "Digikey URL" "https://www.digikey.com/en/products/detail/signal-transformer/F1C1-322510-2R2M/22530386"
 			(at 115.57 78.74 0)
 			(hide yes)
@@
 			)
 		)
-		(property "Manufacturer" ""
+		(property "Manufacturer" "Signal Transformer"
 			(at 115.57 78.74 0)
 			(hide yes)
@@
 			)
 		)
-		(property "Manufacturer Part Number" ""
+		(property "Manufacturer Part Number" "F1C1-322510-2R2M"
 			(at 115.57 78.74 0)
 			(hide yes)
@@
 			)
 		)
-		(property "Datasheet" ""
+		(property "Datasheet" "https://yageogroup.com/content/datasheet/asset/file/UPY-GPHC_X5R_4V-TO-50V"
 			(at 73.66 80.01 0)
 			(hide yes)
@@
 			)
 		)
-		(property "Digikey Part Number" ""
+		(property "Digikey Part Number" "311-3494-2-ND"
 			(at 73.66 80.01 0)
 			(hide yes)
@@
 			)
 		)
-		(property "Digikey URL" ""
+		(property "Digikey URL" "https://www.digikey.com/en/products/detail/yageo/CC0603MRX5R8BB106/7164378?s=N4IgTCBcDaIMwEYEFo4BYCcbkoHIBEQBdAXyA"
 			(at 73.66 80.01 0)
 			(hide yes)
@@
 			)
 		)
-		(property "Manufacturer" ""
+		(property "Manufacturer" " YAGEO"
 			(at 73.66 80.01 0)
 			(hide yes)
@@
 			)
 		)
-		(property "Manufacturer Part Number" ""
+		(property "Manufacturer Part Number" " CC0603MRX5R8BB106"
 			(at 73.66 80.01 0)
 			(hide yes)
@@
 			)
 		)
-		(property "Datasheet" ""
+		(property "Datasheet" "https://1drv.ms/b/c/17a1402ff6a71331/IQCAeqNat8yzR75IgBaxqL_KAZGK2zs81mGDuJqTP0rzcW0?e=wLV0LF"
 			(at 129.54 81.28 0)
 			(hide yes)
@@
 			)
 		)
-		(property "Digikey Part Number" ""
+		(property "Digikey Part Number" "6639-MH0603A226M100N8RCZATR-ND"
 			(at 129.54 81.28 0)
 			(hide yes)
@@
 			)
 		)
-		(property "Digikey URL" ""
+		(property "Digikey URL" "https://www.digikey.com/en/products/detail/sunway-communication/MH0603A226M100N8RCZA/29783836"
 			(at 129.54 81.28 0)
 			(hide yes)
@@
 			)
 		)
-		(property "Manufacturer" ""
+		(property "Manufacturer" "Sunway Communication"
 			(at 129.54 81.28 0)
 			(hide yes)
@@
 			)
 		)
-		(property "Manufacturer Part Number" ""
+		(property "Manufacturer Part Number" "MH0603A226M100N8RCZA"
 			(at 129.54 81.28 0)
 			(hide yes)
