File: pe/timmy-li/actual sch and pcb/buck1.kicad_pcb (KiCad board)
At the start: 2 copper layers, 6 parts, among them U1 TPS62143

Commit message: pcb connection fixes
Parts:
- moved C2 0.50 mm to (116.0, 106.0), turned to 180 degrees
Changed lines of the file:
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@@
 		)
 		(property "Value" "100k"
-			(at 0 1.43 90)
+			(at -3.5 0 180)
 			(layer "F.Fab")
 			(effects
@@
 		(tags "inductor handsolder")
 		(property "Reference" "L1"
-			(at -3 -0.5 180)
+			(at 3 0 180)
 			(layer "F.SilkS")
 			(effects
@@
 		)
 		(property "Value" "2.2uH"
-			(at -4.5 0.5 180)
+			(at -3 0.5 180)
 			(layer "F.Fab")
 			(effects
@@
 	(footprint "Capacitor_SMD:C_0201_0603Metric_Pad0.64x0.40mm_HandSolder"
 		(layer "F.Cu")
-		(at 115.5 106)
+		(at 116 106 180)
 		(descr "Capacitor SMD 0201 (0603 Metric), square (rectangular) end terminal, IPC-7351 nominal with elongated pad for handsoldering. (Body size source: https://www.vishay.com/docs/20052/crcw0201e3.pdf)")
 		(tags "capacitor handsolder")
 		(property "Reference" "C2"
-			(at 0 1.5 180)
+			(at 0 -1.5 0)
 			(layer "F.SilkS")
 			(effects
@@
 		)
 		(property "Value" "22uF"
-			(at 0 3 0)
+			(at 0 -3 0)
 			(layer "F.Fab")
 			(effects
@@
 		)
 		(property "Digikey Part Number" ""
-			(at 0 0 0)
+			(at 0 0 180)
 			(unlocked yes)
 			(layer "F.Fab")
@@
 		)
 		(property "Digikey URL" ""
-			(at 0 0 0)
+			(at 0 0 180)
 			(unlocked yes)
 			(layer "F.Fab")
@@
 		)
 		(property "Manufacturer" ""
-			(at 0 0 0)
+			(at 0 0 180)
 			(unlocked yes)
 			(layer "F.Fab")
@@
 		)
 		(property "Manufacturer Part Number" ""
-			(at 0 0 0)
+			(at 0 0 180)
 			(unlocked yes)
 			(layer "F.Fab")
@@
 		)
 		(pad "" smd roundrect
-			(at -0.4325 0)
+			(at -0.4325 0 180)
 			(size 0.458 0.36)
 			(layers "F.Paste")
@@
 		)
 		(pad "" smd roundrect
-			(at 0.4325 0)
+			(at 0.4325 0 180)
 			(size 0.458 0.36)
 			(layers "F.Paste")
@@
 		)
 		(pad "1" smd roundrect
-			(at -0.4075 0)
+			(at -0.4075 0 180)
 			(size 0.635 0.4)
 			(layers "F.Cu" "F.Mask")
@@
 		)
 		(pad "2" smd roundrect
-			(at 0.4075 0)
+			(at 0.4075 0 180)
 			(size 0.635 0.4)
 			(layers "F.Cu" "F.Mask")

Commit message: moved some stuff
Parts:
- moved C3 1.00 mm to (114.0, 100.0)
- moved C1 0.50 mm to (112.0, 103.5)
- turned L1 to -90 degrees
Changed lines of the file:
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@@
 	(footprint "Capacitor_SMD:C_0201_0603Metric_Pad0.64x0.40mm_HandSolder"
 		(layer "F.Cu")
-		(at 113 100 180)
+		(at 114 100 180)
 		(descr "Capacitor SMD 0201 (0603 Metric), square (rectangular) end terminal, IPC-7351 nominal with elongated pad for handsoldering. (Body size source: https://www.vishay.com/docs/20052/crcw0201e3.pdf)")
 		(tags "capacitor handsolder")
@@
 	(footprint "Capacitor_SMD:C_0201_0603Metric_Pad0.64x0.40mm_HandSolder"
 		(layer "F.Cu")
-		(at 111.5 103.5 -90)
+		(at 112 103.5 -90)
 		(descr "Capacitor SMD 0201 (0603 Metric), square (rectangular) end terminal, IPC-7351 nominal with elongated pad for handsoldering. (Body size source: https://www.vishay.com/docs/20052/crcw0201e3.pdf)")
 		(tags "capacitor handsolder")
@@
 	(footprint "Inductor_SMD:L_1210_3225Metric_Pad1.42x2.65mm_HandSolder"
 		(layer "F.Cu")
-		(at 119.5 104.5 90)
+		(at 119.5 104.5 -90)
 		(descr "Inductor SMD 1210 (3225 Metric), square (rectangular) end terminal, IPC-7351 nominal with elongated pad for handsoldering. (Body size source: http://www.tortai-tech.com/upload/download/2011102023233369053.pdf)")
 		(tags "inductor handsolder")
 		(property "Reference" "L1"
-			(at 3 0 180)
+			(at 3 0 0)
 			(layer "F.SilkS")
 			(effects
@@
 		)
 		(property "Value" "2.2uH"
-			(at -3 0.5 180)
+			(at -3 0 0)
 			(layer "F.Fab")
 			(effects
@@
 		)
 		(property "Digikey Part Number" ""
-			(at 0 0 90)
+			(at 0 0 270)
 			(unlocked yes)
 			(layer "F.Fab")
@@
 		)
 		(property "Digikey URL" ""
-			(at 0 0 90)
+			(at 0 0 270)
 			(unlocked yes)
 			(layer "F.Fab")
@@
 		)
 		(property "Manufacturer" ""
-			(at 0 0 90)
+			(at 0 0 270)
 			(unlocked yes)
 			(layer "F.Fab")
@@
 		)
 		(property "Manufacturer Part Number" ""
-			(at 0 0 90)
+			(at 0 0 270)
 			(unlocked yes)
 			(layer "F.Fab")
@@
 		(duplicate_pad_numbers_are_jumpers no)
 		(fp_line
+			(start -0.602064 1.36)
+			(end 0.602064 1.36)
+			(stroke
+				(width 0.12)
+				(type solid)
+			)
+			(layer "F.SilkS")
+		)
+		(fp_line
 			(start -0.602064 -1.36)
 			(end 0.602064 -1.36)
-			(stroke
-				(width 0.12)
-				(type solid)
-			)
-			(layer "F.SilkS")
-		)
-		(fp_line
-			(start -0.602064 1.36)
-			(end 0.602064 1.36)
 			(stroke
 				(width 0.12)
@@
 		)
 		(pad "1" smd roundrect
-			(at -1.4875 0 90)
+			(at -1.4875 0 270)
 			(size 1.425 2.65)
 			(layers "F.Cu" "F.Mask" "F.Paste")
@@
 		)
 		(pad "2" smd roundrect
-			(at 1.4875 0 90)
+			(at 1.4875 0 270)
 			(size 1.425 2.65)
 			(layers "F.Cu" "F.Mask" "F.Paste")

Commit message: ?? drc
Parts:
- U1: footprint Package_DFN_QFN:VQFN-16-1EP_3x3mm_P0.5mm_EP1.68x1.68mm_ThermalVias -> Package_DFN_QFN:VQFN-16-1EP_3x3mm_P0.5mm_EP1.8x1.8mm_ThermalVias
- moved C2 1.50 mm to (116.0, 107.5)
- moved C1 1.00 mm to (111.0, 103.5)
- moved R1 1.00 mm to (117.0, 100.5)
- moved U1 0.92 mm to (114.9, 103.8)
- moved C3 0.59 mm to (113.4, 100.0)
- moved L1 0.50 mm to (120.0, 104.5)
Connections:
- net Net-(U1-EN) renamed Input 5-17V
- net Net-(U1-VOS) renamed Output 5V/2A
