File: lv/BMS PCB ONBOARDING.kicad_sch (KiCad schematic)
At the start: 75 parts, among them J3 512810598, J4 1053131202, J5 512810598, J6 1053131202, J701 430450200, J702 430450200, Q601 ZXTN4004KTC, U1 BQ79616PAPRQ1

Commit message: UPDATE 3: VC sensing and CB balancing networks drawn
Chip wiring:
- Complete VC1–VC16 cell-tap branches with separate 100Ω sense
  resistors and 10Ω balancing resistors
- Add 0.47uF differential capacitors from VC16–VC15 through VC1–VC0
- Connect VC0 to cell 1 negative through 100Ω, with a chip-side
  0.47uF capacitor to AVSS
- Connect CB0–CB16 chip pins to matching balancing resistor nets
  using bidirectional global labels
- Add 0.47uF differential capacitors from CB16–CB15 through CB1–CB0
- Connect CB0 to cell 1 negative through 10Ω, with a chip-side
  0.47uF capacitor to AVSS
- Add the extra 470nF capacitor between CB16 and BAT 

Blocks on the sheet:
- Add the ZXTN25100DGTA due to old circuit not having enough voltage
   for LDOIN
- Correct VC capacitors from series placement to differential wiring
- Add direct CB pin-net connections before the filter capacitors
- Correct the CB0 resistor branch to the raw cell-negative VC0 net

Pending:
- Confirm cell voltage, balancing-current target and balancing mode
- Verify resistor values, power ratings and derating
- Finalize capacitor ratings and footprints
- Run annotation, ERC and netlist connectivity checks

Learned:
- Internal balancing FETs handle the balancing circuit meaning 
   we don't need any balancing blocks
- Filter capacitors belong between adjacent chip-side nodes
- VC0 and CB0 need separate resistor paths from cell 1
- CB16–BAT requires an additional capacitor, not a replacement
  for CB16–CB15
- 470nF equals 0.47uF
- Balancing resistance and power ratings must be checked together
- TSREF does not replace LDOIN supply conditioning
Parts:
- removed C601: 0.22uF, GCM31MR72A224KA37L:G-31_MUR-L, symbol GCM31MR72A224KA37L:GCM31MR72A224KA37L
- removed Q601: ZXTN4004KTC, ZXTN4004KTC:ZXTN4004KTC, symbol ZXTN4004KTC:ZXTN4004KTC
- removed R601: 100, CRCW2010100RFKEF:RES_CRCW_2010-L, symbol CRCW2010100RFKEF:CRCW2010100RFKEF
- removed R602: 200, Resistor_SMD:R_2512_6332Metric, symbol CRCW2010200RFKEF:CRCW2010200RFKEF
- added C1, C10, C11, C12, C19, C2, C20, C21, C22, C24, C25, C26, C27, C28, C29, C3, C30, C31, C32, C33, C34, C35, C36, C37, C38, C39, C4, C40, C5, C6, C7, C8, C9: .47uF, symbol Device:C
- added C41: 470nF, symbol Device:C
- added C602: 0.22uF, GCM31MR72A224KA37L:G-31_MUR-L, symbol GCM31MR72A224KA37L:GCM31MR72A224KA37L
- added Q1: ZXTN25100DGTA, SOT223_DIO, symbol 2026-10-10_18-40-02:ZXTN25100DGTA
- added R100, R102, R103, R117, R119, R122, R123, R124, R80, R83, R86, R87, R91, R92, R94, R96, R98: 100, Resistor_SMD:R_0805_2012Metric_Pad1.20x1.40mm_HandSolder, symbol Device:R
- added R101, R116, R118, R120, R121, R125, R81, R82, R84, R85, R88, R89, R90, R93, R95, R97, R99: 10, Resistor_SMD:R_0805_2012Metric_Pad1.20x1.40mm_HandSolder, symbol Device:R
- added R603: 100, CRCW2010100RFKEF:RES_CRCW_2010-L, symbol CRCW2010100RFKEF:CRCW2010100RFKEF
- added R604: 200, Resistor_SMD:R_2512_6332Metric, symbol CRCW2010200RFKEF:CRCW2010200RFKEF
Connections:
- net BAT: now also C41.2, R604.2, R80.1, R81.1; no longer U1.3 (VC16)
- net CB0: now also C32.2, C40.2, R125.1
- net CB1: now also C32.1, C33.2, R120.2
- net CB10: now also C29.1, C30.2
- net CB11: now also C30.1, C31.2, R90.2
- net CB12: now also C26.2, C31.1, R84.2
- net CB13: now also C26.1, C27.2, R85.2
- net CB14: now also C25.2, C27.1, R89.2
- net CB15: now also C24.2, C25.1, R82.2
- net CB16: now also C24.1, C41.1, R81.2
- net CB2: now also C33.1, C34.2, R121.2
- net CB3: now also C34.1, C35.2, R118.2
- net CB4: now also C35.1, C36.2, R116.2
- net CB5: now also C36.1, C37.2, R93.2
- net CB6: now also C37.1, C38.2, R88.2
- net CB7: now also C38.1, C39.2, R95.2
- net CB8: now also C28.2, C39.1, R97.2
- net CB9: now also C28.1, C29.2, R99.2
- net CVDD: now also U1.52 (RX)
- net GND: now also C21.1, C40.1, C602.2
- net LDOIN: now also Q1.2, Q1.3
- net NPNB: now also Q1.1
- net VC0: now also R124.1, R125.2; no longer U1.35 (VC0)
- net VC1: now also R120.1, R122.1; no longer U1.33 (VC1)
- net VC10: now also R101.1, R103.1; no longer U1.15 (VC10)
- net VC11: now also R90.1, R92.1; no longer U1.13 (VC11)
- net VC12: now also R84.1, R86.1; no longer U1.11 (VC12)
- net VC13: now also R85.1, R87.1; no longer U1.9 (VC13)
- net VC14: now also R89.1, R91.1; no longer U1.7 (VC14)
- net VC15: now also R82.1, R83.1; no longer U1.5 (VC15)
- net VC2: now also R121.1, R123.1; no longer U1.31 (VC2)
- net VC3: now also R118.1, R119.1; no longer U1.29 (VC3)
- net VC4: now also R116.1, R117.1; no longer U1.27 (VC4)
- net VC5: now also R93.1, R94.1; no longer U1.25 (VC5)
- net VC6: now also R88.1, R96.1; no longer U1.23 (VC6)
- net VC7: now also R95.1, R98.1; no longer U1.21 (VC7)
- net VC8: now also R100.1, R97.1; no longer U1.19 (VC8)
- net VC9: now also R102.1, R99.1; no longer U1.17 (VC9)
- new net: C5.1, C8.2, R94.2, U1.25 (VC5)
- new net: C5.2, C9.1, R96.2, U1.23 (VC6)
- new net: C20.1, C22.2, R123.2, U1.31 (VC2)
- new net: C22.1, R122.2, U1.33 (VC1)
- new net: C1.1, C2.2, R83.2, U1.5 (VC15)
- new net: C1.2, R80.2, U1.3 (VC16)
- new net: C602.1, Q1.4, R603.2
- new net: R603.1, R604.1
- new net: C10.1, C9.2, R98.2, U1.21 (VC7)
- new net: C3.2, C4.1, R86.2, U1.11 (VC12)
- new net: C10.2, C11.1, R100.2, U1.19 (VC8)
- new net: C11.2, C12.1, R102.2, U1.17 (VC9)
- new net: C19.1, C20.2, R119.2, U1.29 (VC3)
- new net: C19.2, C8.1, R117.2, U1.27 (VC4)
- new net: C3.1, C7.2, R92.2, U1.13 (VC11)
- new net: C4.2, C6.1, R87.2, U1.9 (VC13)
- new net: C21.2, R124.2, U1.35 (VC0)
- new net: C12.2, C7.1, R103.2, U1.15 (VC10)
- new net: C2.1, C6.2, R91.2, U1.7 (VC14)
- no-connect marks 7 -> 6
Other:
- note added: "ALL CAPS IN CB CIRCUT ARE .47uF"
- moved on the sheet: TP509

Commit message: UPDATE 4: ERC and footprint cleanup complete, schematic closed for routing
Chip wiring:
- Connect R101 pin 2 to CB10 with global label,
  cell-10 balance path now complete
- Remove dead VREG net, re-point R9/R12/R14 pull-ups
  to driven TSREF rail
- Add 0.47uF differential capacitor VC1-VC0 (C23),
  all 16 VC rungs + VC0-AVSS now present
- Verify complete CB ladder: 16 rungs + CB0-AVSS
  + CB16-BAT (34x 0.47uF + 470nF C41)
- Delete unconnected R43 and TP1,
  only intentional NCs remain
- Correct Q1 ZXTN25100DGTA emitter-follower: move pin 2
  collector lead from LDOIN to pin-4 feed junction
  (C602/R603), pin 3 emitter to LDOIN, pin 1 base to NPNB
- Fix C207 DVDD value to 2.2uF with correct 2.2uF MPN

Blocks on the sheet:
- Move Q1 pin-2 wire from LDOIN label to C602/R603 junction
- Delete duplicate PWR_FLAG #FLG01 after VREG merge into TSREF,
  clear NEG5V pin-type exclusion, ERC now zero errors
- Assigned all 42 missing footprints, move 17x 10R balancers
  to 2512 1W, fix R604 / C207 / C701-C708 / FL701-FL702 libs
- Register footprint libs, Update PCB from Schematic loads clean
- Run annotation, ERC and netlist connectivity checks clean

Pending:
- PCB routing only, schematic closed
- Place VC/CB filter block tight to U1, then power,
  then comms daisy-chain
- Set 67V clearance/creepage rules before routing taps
- Run DRC and copper-balance check for 10R heat

Learned:
- ERC clean does not mean electrically correct,
  Q1 C-E short and C207 MPN mismatch are invisible to ERC
- Pins 2 + 4 on ZXTN25100DGTA are both collector (lead + tab),
  splitting them shorts C-E through the part
- Renaming VREG to TSREF merges PWR_FLAGs onto one net,
  the old flag must be deleted
- Filter capacitors belong between adjacent chip-side nodes,
  VC0 and CB0 need separate resistor paths from cell 1
- Balancing resistance and power ratings must be checked together,
  10R needs 2512 1W not 0805
Parts:
- removed R43: 1K, Resistor_SMD:R_0603_1608Metric_Pad0.98x0.95mm_HandSolder, symbol Device:R
- removed TP1: S6, TestPoint:TestPoint_Pad_D1.5mm, symbol Connector:TestPoint
- added C23: .47uF, Capacitor_SMD:C_0603_1608Metric, symbol Device:C
- C1, C10, C11, C12, C19, C2, C20, C21, C22, C24, C25, C26, C27, C28, C29, C3, C30, C31, C32, C33, C34, C35, C36, C37, C38, C39, C4, C40, C41, C5, C6, C7, C8, C9: footprint (none) -> Capacitor_SMD:C_0603_1608Metric
- C207: value 2.2.uF -> 2.2uF
- Q1: footprint SOT223_DIO -> footprintsZXTN25100DGTA:SOT223_DIO
- R1, R2, R3, R4, R5, R7, R8: footprint (none) -> Resistor_SMD:R_0805_2012Metric
- R101, R116, R118, R120, R121, R125, R81, R82, R83, R84, R85, R88, R89, R90, R93, R95, R97, R99: footprint Resistor_SMD:R_0805_2012Metric_Pad1.20x1.40mm_HandSolder -> Resistor_SMD:R_2512_6332Metric
- R604: footprint Resistor_SMD:R_2512_6332Metric -> Resistor_SMD:R_2010_5025Metric
- U1: footprint PAP0064F-IPC_A -> footprintsBQ79616PAPRQ1:PAP0064F-IPC_A
Connections:
- net VREG is gone; now on net TSREF: R12.1, R14.1, R9.1
- net CB10: now also R101.2
- net LDOIN: no longer Q1.2
- net at C22.1, R122.2, U1.33 (VC1): now also C23.2
- net at C602.1, Q1.4, R603.2: now also Q1.2
- net at C21.2, R124.2, U1.35 (VC0): now also C23.1
