File: pe/maheer-grang/maheer-grang.kicad_sch (KiCad schematic)
At the start: 0 parts

Commit message: finished lv project research, working on lv board schematic. worked on pe buck schematic
Parts:
- added C1, C2, C3, C4, C5: C_Small, symbol Device:C_Small
- added L1: L_Small, symbol Device:L_Small
- added R1, R2, R3, R4: R_Small_US, symbol Device:R_Small_US
- added U1: AP62300TWU, Package_TO_SOT_SMD:TSOT-23-6, symbol Regulator_Switching:AP62300TWU
Connections:
- new net: C1.1, C2.1, R1.1, U1.3 (IN)
- new net: C4.1, C5.1, L1.2, R3.1
- new net: R3.2, R4.1, U1.4 (FB)
- new net: C3.2, L1.1, U1.2 (SW)
- new net: R1.2, R2.1, U1.5 (EN)
- new net: C3.1, U1.6 (BST)
- new net GNDREF: C1.2, C2.2, C4.2, C5.2, R2.2, R4.2, U1.1 (GND)

Commit message: finished schematic, working on pcb design
Parts:
- C1, C2: value C_Small -> 10 µF; footprint (none) -> Capacitor_SMD:C_1206_3216Metric; Digikey Part Number (none) -> 490-6518-1-ND; Digikey URL (none) -> https://www.digikey.com/en/products/detail/murata-electroni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; Manufacturer (none) -> Murata Electronics; Manufacturer Part Number (none) -> GRM31CR71E106KA12L
- C3: value C_Small -> 100 nF; footprint (none) -> Capacitor_SMD:C_0603_1608Metric_Pad1.08x0.95mm_HandSolder; Digikey Part Number (none) -> 311-1344-1-ND; Digikey URL (none) -> https://www.digikey.com/en/products/detail/yageo/CC0603KRX7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; Manufacturer (none) -> YAGEO; Manufacturer Part Number (none) -> CC0603KRX7R9BB104
- C4, C5: value C_Small -> 22 µF; footprint (none) -> Capacitor_SMD:C_0603_1608Metric_Pad1.08x0.95mm_HandSolder; Digikey Part Number (none) -> 478-KGM15CR51C226MTCT-ND; Digikey URL (none) -> www.digikey.com/en/products/detail/kyocera-avx/0603YD226MAT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; Manufacturer (none) -> KYOCERA AVX; Manufacturer Part Number (none) -> 0603YD226MAT2A
- L1: value L_Small -> B82464P4472M000; footprint (none) -> Inductor_SMD:L_10.4x10.4_H4.8; Digikey Part Number (none) -> 495-77086-1-ND; Manufacturer (none) -> TDK; Manufacturer Part Number (none) -> B82464P4472M000
- R1: value R_Small_US -> 56.2k; footprint (none) -> Resistor_SMD:R_0603_1608Metric_Pad0.98x0.95mm_HandSolder; Digikey Part Number (none) -> 311-56.2KHRCT-ND; Digikey URL (none) -> https://www.digikey.com/en/products/detail/yageo/RC0603FR-0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; Manufacturer (none) -> YAGEO; Manufacturer Part Number (none) -> RC0603FR-0756K2L
- R2: value R_Small_US -> 10K; footprint (none) -> Resistor_SMD:R_0603_1608Metric_Pad0.98x0.95mm_HandSolder; Digikey Part Number (none) -> 311-10KLDCT-ND; Digikey URL (none) -> https://www.digikey.com/en/products/detail/yageo/AC0603FR-0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; Manufacturer (none) -> YAGEO; Manufacturer Part Number (none) -> AC0603FR-0710KL
- R3: value R_Small_US -> 221K; footprint (none) -> Resistor_SMD:R_0603_1608Metric_Pad0.98x0.95mm_HandSolder; Digikey Part Number (none) -> 13-AC0603FR-07221KLCT-ND; Digikey URL (none) -> https://www.digikey.com/en/products/detail/yageo/AC0603FR-0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; Manufacturer (none) -> YAGEO; Manufacturer Part Number (none) -> AC0603FR-07221KL
- R4: value R_Small_US -> 32.4K; footprint (none) -> Resistor_SMD:R_0603_1608Metric_Pad0.98x0.95mm_HandSolder; Digikey Part Number (none) -> 13-AC0603FR-0732K4LCT-ND; Digikey URL (none) -> https://www.digikey.com/en/products/detail/yageo/AC0603FR-0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; Manufacturer (none) -> YAGEO; Manufacturer Part Number (none) -> AC0603FR-0732K4L
Connections:
- net at C1.1, C2.1, U1.3 (IN): now also R3.1; no longer R1.1
- net at C4.1, C5.1, L1.2: now also R1.1; no longer R3.1
- net at R3.2, R4.1: now also U1.5 (EN); no longer U1.4 (FB)
- net at R1.2, R2.1: now also U1.4 (FB); no longer U1.5 (EN)
Other:
- title: ${BOARD_TITLE} -> PE Buck Converter Onboarding Project
