File: pe/12V-buck/12V-buck.kicad_sch (KiCad schematic)
At the start: 0 parts

Commit message: 12V Schem
Parts:
- added C1: 10uF, Capacitor_SMD:C_0603_1608Metric_Pad1.08x0.95mm_HandSolder, symbol Device:C
- added C2: 100nF, Capacitor_SMD:C_0603_1608Metric_Pad1.08x0.95mm_HandSolder, symbol Device:C
- added C3, C4: 22uF, Capacitor_SMD:C_0603_1608Metric_Pad1.08x0.95mm_HandSolder, symbol Device:C
- added L1: 3.3uH, Inductor_SMD:L_Bourns_SRN6045TA, symbol Device:L
- added R1: 100k, Resistor_SMD:R_0603_1608Metric_Pad0.98x0.95mm_HandSolder, symbol Device:R_US
- added R2: 10k, Resistor_SMD:R_0603_1608Metric_Pad0.98x0.95mm_HandSolder, symbol Device:R_US
- added R3: 54.9k, Resistor_SMD:R_0603_1608Metric_Pad0.98x0.95mm_HandSolder, symbol Device:R_US
- added U1: TPS563208, Package_TO_SOT_SMD:SOT-23-6, symbol Regulator_Switching:TPS563208
Connections:
- new net: R2.1, R3.1, U1.4 (VFB)
- new net: C2.1, L1.1, U1.2 (SW)
- new net: R1.2, U1.5 (EN)
- new net: C2.2, U1.6 (VBST)
- new net +12V: C1.1, R1.1, U1.3 (VIN)
- new net +5V: C3.1, C4.1, L1.2, R3.2
- new net GND: C1.2, C3.2, C4.2, R2.2, U1.1 (GND)
