File: pe/kicad-template/template.kicad_sch (KiCad schematic)
At the start: 4 parts

Commit message: Update docs
Parts:
- L1: value 10.5uH -> 12uH
Connections:
- net V_in 13.5v renamed V_in 15v
Changed lines of the file:
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@@
 		)
 	)
-	(label "V_in 13.5v"
+	(label "V_in 15v"
 		(at 67.31 83.82 0)
 		(effects
@@
 			)
 		)
-		(property "Value" "10.5uH"
+		(property "Value" "12uH"
 			(at 125.73 67.31 90)
 			(show_name no)

Commit message: update parts
Parts:
- removed R1: R_Load, symbol Device:R_Small
- C1: value 15uF -> 22uF; Digikey Part Number (none) -> 4713-GMC10X5R226M10NTDKR-ND; Digikey URL (none) -> https://www.digikey.com/en/products/detail/cal-chip-electro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; Manufacturer (none) -> Cal-Chip Electronics, Inc.; Manufacturer Part Number (none) -> GMC10X5R226M10NT
- L1: value 12uH -> 15uH; Digikey Part Number (none) -> 283-SDCHA1V8040-150-RDKR-ND; Digikey URL (none) -> https://www.digikey.com/en/products/detail/eaton-electronic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; Manufacturer (none) -> Eaton - Electronics Division; Manufacturer Part Number (none) -> SDCHA1V8040-150-R
- U1: value (none) -> TPS542025DDCR; Digikey Part Number (none) -> 296-TPS542025DDCRDKR-ND; Digikey URL (none) -> https://www.digikey.com/en/products/detail/texas-instrument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; Manufacturer (none) -> Texas Instruments; Manufacturer Part Number (none) -> TPS542025DDCR
Connections:
- net GND is gone; now on net +5V: C1.2, U1.1 (GND)
- net +5V: now reaches C1.1, L1.2
- net V_in 15v renamed +15V
