File: pe/kicad-template/template.kicad_sch (KiCad schematic)
At the start: 0 parts

Commit message: some first files, likely to change later, plus some of the example project in that kicad workshop
Parts:
- added C1: 10nF, Capacitor_SMD:CP_Elec_6.3x3, symbol KiCad:C_Small
- added C2: C0603C104M3VACTU, capacitor:CAPC1608X90N, symbol capacitor:C0603C104M3VACTU
- added D1: D_Small, Diode_SMD:D_0201_0603Metric, symbol KiCad:D_Small
- added IC1: TS30013-M050QFNR, QFN50P300X300X100-17N-D, symbol outside_symbols:TS30013-M050QFNR
- added J1: Conn_01x02, Connector_PinSocket_2.54mm:PinSocket_1x06_P2.54mm_Vertical, symbol KiCad:Conn_01x02
- added J2: PK_HOLD_OUT, Connector_PinSocket_2.54mm:PinSocket_1x06_P2.54mm_Vertical, symbol KiCad:Conn_01x02
- added R1: 24k, Resistor_SMD:R_0603_1608Metric, symbol KiCad:R_Small
- added R2: 1k, Resistor_SMD:R_0603_1608Metric, symbol KiCad:R_Small
- added U1: MCP6004, formula_slug_footprint_library:SOIC-8_ISO1044BD, symbol KiCad:MCP6004
Connections:
- new net: R1.1, R2.1, U1.3 (+)
- new net: J1.2 (Pin_2), R1.2
- new net: C1.1, D1.1 (K), U1.2 (-), U1.5 (+)
- new net: J2.1 (Pin_1), U1.6 (-), U1.7
- new net: D1.2 (A), U1.1
- new net GND: C1.2, J1.1 (Pin_1), J2.2 (Pin_2), R2.2
