File: pe/Buck-Converter-Design/template.kicad_pcb (KiCad board)
At the start: 2 copper layers, 21.5 x 17 mm, 7 parts, among them U1 TPS562200

Commit message: PE KiCad notes
Did a lot for PE involving taking more in depth notes with visuals of how thigns work so I can more deeply understand them.
Parts:
- moved C1 2.29 mm to (127.7, 114.0)
- moved R2 1.18 mm to (114.1, 117.0)
Routing:
- net GND: track 41.5 -> 36.5 mm
- net Net-(U1-VFB): track 11.9 -> 9.58 mm
Changed lines of the file:
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@@
 	(footprint "Resistor_SMD:R_0805_2012Metric"
 		(layer "F.Cu")
-		(at 112.9125 117)
+		(at 114.0875 117)
 		(descr "Resistor SMD 0805 (2012 Metric), square (rectangular) end terminal, IPC-7351 nominal, (Body size source: IPC-SM-782 page 72, https://www.pcb-3d.com/wordpress/wp-content/uploads/ipc-sm-782a_amendment_1_and_2.pdf)")
 		(tags "resistor")
@@
 	(footprint "Capacitor_SMD:C_1210_3225Metric"
 		(layer "F.Cu")
-		(at 129.5 112.525 -90)
+		(at 127.725 113.975 -90)
 		(descr "Capacitor SMD 1210 (3225 Metric), square (rectangular) end terminal, IPC-7351 nominal, (Body size source: IPC-SM-782 page 76, https://www.pcb-3d.com/wordpress/wp-content/uploads/ipc-sm-782a_amendment_1_and_2.pdf)")
 		(tags "capacitor")
@@
 	)
 	(gr_rect
-		(start 110 104.5)
-		(end 131.5 121.5)
+		(start 108.225 105.95)
+		(end 129.725 122.95)
 		(stroke
 			(width 0.0508)
@@
 	)
 	(segment
+		(start 123.094 120.081)
+		(end 118.469204 120.081)
+		(width 0.254)
+		(layer "F.Cu")
+		(net "GND")
+	)
+	(segment
+		(start 118.469204 117.919)
+		(end 118.5 117.919)
+		(width 0.254)
+		(layer "F.Cu")
+		(net "GND")
+	)
+	(segment
 		(start 122.356 114.982248)
 		(end 122.356 112.467752)
@@
 	)
 	(segment
-		(start 129.5 114)
-		(end 123.419 120.081)
+		(start 115 117)
+		(end 117.581 117)
+		(width 0.254)
+		(layer "F.Cu")
+		(net "GND")
+	)
+	(segment
+		(start 117.581 117)
+		(end 118.5 117.919)
+		(width 0.254)
+		(layer "F.Cu")
+		(net "GND")
+	)
+	(segment
+		(start 118.1065 118.281704)
+		(end 118.469204 117.919)
+		(width 0.254)
+		(layer "F.Cu")
+		(net "GND")
+	)
+	(segment
+		(start 118.1065 119.718296)
+		(end 118.1065 118.281704)
 		(width 0.254)
 		(layer "F.Cu")
@@
 	)
 	(segment
-		(start 118.1065 118.281704)
-		(end 118.469204 117.919)
-		(width 0.254)
-		(layer "F.Cu")
-		(net "GND")
-	)
-	(segment
-		(start 120.338248 117)
-		(end 113.825 117)
-		(width 0.254)
-		(layer "F.Cu")
-		(net "GND")
-	)
-	(segment
 		(start 118.469204 120.081)
 		(end 118.1065 119.718296)
@@
 	)
 	(segment
-		(start 118.469204 117.919)
-		(end 119.419248 117.919)
-		(width 0.254)
-		(layer "F.Cu")
-		(net "GND")
-	)
-	(segment
-		(start 118.1065 119.718296)
-		(end 118.1065 118.281704)
-		(width 0.254)
-		(layer "F.Cu")
-		(net "GND")
-	)
-	(segment
-		(start 123.419 120.081)
-		(end 118.469204 120.081)
-		(width 0.254)
-		(layer "F.Cu")
-		(net "GND")
-	)
-	(segment
 		(start 119.281 112.119)
 		(end 118.9 112.5)
@@
 	)
 	(segment
+		(start 118.5 117.919)
+		(end 119.419248 117.919)
+		(width 0.254)
+		(layer "F.Cu")
+		(net "GND")
+	)
+	(segment
 		(start 119.5 108)
 		(end 119.5 111.9)
@@
 	)
 	(segment
-		(start 114.225 114.775)
+		(start 127.725 115.45)
+		(end 123.094 120.081)
+		(width 0.254)
+		(layer "F.Cu")
+		(net "GND")
+	)
+	(segment
+		(start 113.175 117)
+		(end 115.175 119)
+		(width 0.254)
+		(layer "F.Cu")
+		(net "Net-(U1-VFB)")
+	)
+	(segment
+		(start 115.4 114.775)
 		(end 117 114.775)
 		(width 0.254)
@@
 	)
 	(segment
-		(start 112 117)
-		(end 114 119)
+		(start 115.175 119)
+		(end 117.175 119)
 		(width 0.254)
 		(layer "F.Cu")
@@
 	)
 	(segment
-		(start 112 117)
-		(end 114.225 114.775)
-		(width 0.254)
-		(layer "F.Cu")
-		(net "Net-(U1-VFB)")
-	)
-	(segment
-		(start 114 119)
-		(end 117.175 119)
+		(start 113.175 117)
+		(end 115.4 114.775)
 		(width 0.254)
 		(layer "F.Cu")
@@
 	)
 	(segment
-		(start 125.5 108.5)
-		(end 128.05 111.05)
-		(width 0.254)
-		(layer "F.Cu")
-		(net "/VOUT")
-	)
-	(segment
 		(start 119 119)
 		(end 119.5125 119)
@@
 	)
 	(segment
-		(start 128.05 111.05)
-		(end 129.5 111.05)
-		(width 0.254)
-		(layer "F.Cu")
+		(start 125.5 110.275)
+		(end 125.5 108.5)
+		(width 0.254)
+		(layer "F.Cu")
+		(net "/VOUT")
+	)
+	(segment
+		(start 127.725 112.5)
+		(end 125.5 110.275)
+		(width 0.254)
+		(layer "F.Cu")
