File: pe/Buck-Converter-Design/template.kicad_sch (KiCad schematic)
At the start: 7 parts, among them U1 TPS562200

Commit message: PE KiCad notes
Did a lot for PE involving taking more in depth notes with visuals of how thigns work so I can more deeply understand them.
Parts:
- added BT1: Input, Package_SON:Texas_DRC0010J_ThermalVias, symbol Device:Battery_Cell
- added C4: C Smooth, symbol Device:C
- added C5: C Smooth, Package_DIP:DIP-8_W7.62mm, symbol Device:C
- added Q1: BSS308PE, Package_TO_SOT_SMD:SOT-23_Handsoldering, symbol formula_slug_symbol_library:BSS308PE
- added R3: Output, symbol Device:R
- added U2: TPS562200, Package_TO_SOT_SMD:SOT-23-6, symbol Regulator_Switching:TPS562200
Connections:
- new net: BT1.2 (-), C4.2, C5.2, Q1.1 (G), R3.2
- new net: C5.1, Q1.2 (S), R3.1
- new net: BT1.1 (+), C4.1, Q1.3 (D)
Other:
- note added: "Bootstrap Capactiro connected to VBST to give constant supply of power to the switching device"
- note added: "Bootstrap capacitor store Vin and then + the stored capactiro voltage"
- note added: "Bootstrap: connects to SW through a bootstrap capacitor to keep a higher voltage than Vin to drive the gate to the MOSFET switch"
- note added: "Enable pin: keeps the regulator on"
- note added: "Ground"
- note added: "Input"
- note added: "Input voltage"
- note added: "MOSFET switch output"
- note added: "Power Stepdown"
- note added: "Smooths the current"
- note added: "Stabalize output voltage"
- note added: "Voltage Feedback: Monitor and regulate the output voltage. It measures based off a internal reference. The converter adjusts the duty cycle to reach the intended output voltage"
- note added: "stabalize input voltage"
- note added: "used to give buck converter able to see output voltage to make sure its at the steady target voltage"
- moved on the sheet: C1, C2, C3, L1, R1, R2, U1
