File: lv/Comparator Kicad/template.kicad_sch (KiCad schematic)
At the start: 5 parts, among them U1 LM397

Commit message: LV Schematic Notes
Trying to understand the comaprator and Op-Amp more deeply thorugh the schematics with notes
Parts:
- added U2: LM397, Package_TO_SOT_SMD:SOT-23-5, symbol Comparator:LM397
Other:
- note added: "Negative Supply / GND: connects to ground for the negative power rail for the IC"
- note added: "Out1: Either connects the ouput pin directly to ground or leaves the pin unpowered"
- note added: "Positive Supply: powers the comparator"
- note added: "VIN1: Non-Inverting Input voltage that gets evauated"
- note added: "VREF1: reference voltage to be the level against which the input is measured"
- note added: "When the internal transistor is turned off, there is no current flowing so there is no voltage drop across teh resisstor so 5V When the internal transistor is turned on, Current flows through thte resisitor and transistior to ground, the output drops to a low voltage"
- moved on the sheet: OUT1, Pull-up1, U1, VIN1, VREF1
