File: lv/Op-Amp Kicad/template.kicad_sch (KiCad schematic)
At the start: 3 parts, among them U1 ${SIM.PARAMS}

Commit message: LV Schematic Notes
Trying to understand the comaprator and Op-Amp more deeply thorugh the schematics with notes
Parts:
- added Out1: Conn_01x01, Connector:Tag-Connect_TC2030-IDC-FP_2x03_P1.27mm_Vertical, symbol Connector_Generic:Conn_01x01
Connections:
- net at R1.2, U1.5: now also Out1.1 (Pin_1)
Other:
- note added: "2.5V reference voltage"
- note added: "5V postitive power supply"
- note added: "Ground"
- note added: "Output current"
- note added: "When the ouput trasnsistor is off, the reiistors create a higher upper switchign threshold, adn when teh ouput transissor is on, they create a lower lower switchign threshold"
- note added: "having input current be AC has the comaprator switch from high to low often meaning the comaprator switches constantly"
- moved on the sheet: R1, R2, U1
